File: SunBladeNVRAM.kicad_sch (KiCad schematic)
At the start: 15 parts, among them J1 Conn_01x14_Pin, J105 Conn_01x01_Pin, J106 Conn_01x01_Pin, J107 Conn_01x01_Pin, J108 Conn_01x01_Pin, J2 Conn_01x14_Pin, J3 Conn_01x02_Pin, J4 Conn_01x02_Pin, J5 Conn_01x01_Pin, J6 Conn_01x01_Pin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

Commit message: improved 1x14 header, M48T59Y-MH footprints
The 1x14 header footprint is for round (machine pin)
headers, which is what we want to use. The through holes
are much more compact than the footprint for normal
square headers.

The M48T59Y footprint is made slightly more compact.
It should still allow plenty of room to solder on the
M49T59Y, but it fits relatively comfortably between
the 1x14 pin headers.

With these changes, it shouldn't be necessary to bend
the legs of the M48T59Y.
Parts:
- J1, J2: footprint Connector_PinHeader_2.54mm:PinHeader_1x14_P2.54mm_Vertical -> SunBladeNVRAM:SAMTEC_BBL-114-T-E
- U1: footprint Package_SO:SOIC-28W_7.5x17.9mm_P1.27mm -> SunBladeNVRAM:M48T59Y-MH
Changed lines of the file:
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@@
 			)
 		)
-		(property "Footprint" "Connector_PinHeader_2.54mm:PinHeader_1x14_P2.54mm_Vertical"
+		(property "Footprint" "SunBladeNVRAM:SAMTEC_BBL-114-T-E"
 			(at 44.45 78.74 0)
 			(effects
@@
 			)
 		)
-		(property "Footprint" "Connector_PinHeader_2.54mm:PinHeader_1x14_P2.54mm_Vertical"
+		(property "Footprint" "SunBladeNVRAM:SAMTEC_BBL-114-T-E"
 			(at 123.19 78.74 0)
 			(effects
@@
 			)
 		)
-		(property "Footprint" "Package_SO:SOIC-28W_7.5x17.9mm_P1.27mm"
+		(property "Footprint" "SunBladeNVRAM:M48T59Y-MH"
 			(at 83.82 80.01 0)
 			(effects
