File: SunBladeNVRAM.kicad_pcb (KiCad board)
At the start: 2 copper layers, 36.5 x 18.5 mm, 10 parts, among them J1 Conn_01x14_Pin, J2 Conn_01x14_Pin, J3 Conn_01x02_Pin, J4 Conn_01x02_Pin, J5 Conn_01x01_Pin, J6 Conn_01x01_Pin, J7 Conn_01x01_Pin, J8 Conn_01x01_Pin, U1 M48T59Y-70MH1, Y1 32.768 kHz

Commit message: routed all traces, a few minor tweaks
Ready to fab?
Routing:
- net Net-(J1-Pin_1): track 0.00 -> 15.7 mm, vias 0 -> 1
- net Net-(J1-Pin_2): track 0.00 -> 14.7 mm, vias 0 -> 1
- net Net-(J2-Pin_2): track 0.00 -> 14.5 mm, vias 0 -> 1
- net Net-(J2-Pin_1): track 0.00 -> 13.6 mm
- net Net-(J2-Pin_3): track 0.00 -> 13.5 mm, vias 0 -> 1
- net Net-(J1-Pin_3): track 0.00 -> 13.2 mm, vias 0 -> 1
- net Net-(J2-Pin_4): track 0.00 -> 11.9 mm, vias 0 -> 1
- net Net-(J1-Pin_4): track 0.00 -> 11.9 mm, vias 0 -> 1
- net Net-(J1-Pin_5): track 0.00 -> 10.6 mm, vias 0 -> 1
- net Net-(J2-Pin_5): track 0.00 -> 10.6 mm, vias 0 -> 1
- net Net-(J2-Pin_6): track 0.00 -> 9.38 mm, vias 0 -> 1
- net Net-(J1-Pin_6): track 0.00 -> 9.37 mm, vias 0 -> 1
- net Net-(J2-Pin_7): track 0.00 -> 8.14 mm, vias 0 -> 1
- net Net-(J1-Pin_7): track 0.00 -> 8.11 mm, vias 0 -> 1
- net Net-(J1-Pin_8): track 0.00 -> 7.13 mm, vias 0 -> 1
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Other:
- board text added: "Sun Blade 150 NVRAM replacement (c) 2024, daveho hacks https://github.com/daveho/SunBladeNVRAM Revision 2, 10-Dec-2024"
- board text removed: "Sun Blade 150 NVRAM replacement (c) 2024, daveho hacks https://github.com/daveho/SunBladeNVRAM"
